Commit message: updating gazebo config for ardrone

File: usma_descriptions/UAV/urdf/usma_ardrone_base.urdf.xacro (robot description, xacro)
@@ -1,7 +1,7 @@
 <robot xmlns:xacro="http://ros.org/wiki/xacro">
   <xacro:property name="X_ROBOT_NAMESPACE" value="/gazebo/uav" />
-  <xacro:include filename="$(find robot_plugins)/urdf/ardrone_plugins.urdf.xacro" />
+  <xacro:include filename="$(find usma_plugins)/urdf/usma_ardrone_plugins.urdf.xacro" />
   <!-- Main ardrone link -->
-  <xacro:macro name="ardrone_base_macro">
+  <xacro:macro name="usma_ardrone_base_macro">
 	<link name="${X_ROBOT_NAMESPACE}/ardrone_base_footprint"/>
 	<joint name="base_joint" type="fixed">
@@ -29,32 +29,9 @@
       </collision>
     </link>
-  <!-- LEDs -->
-    <xacro:include filename="$(find robot_descriptions)/UAV/urdf/link_led.urdf.xacro" />
-    <!-- Red -->
-        <xacro:link_led name="${X_ROBOT_NAMESPACE}/ardrone_red" parent="${X_ROBOT_NAMESPACE}/ardrone_base_link">
-          <origin xyz="0.0 -0.22 -0.01" rpy="0 0 0"/>
-        </xacro:link_led>
-    <!-- Blue -->
-        <xacro:link_led name="${X_ROBOT_NAMESPACE}/ardrone_blue" parent="${X_ROBOT_NAMESPACE}/ardrone_base_link">
-          <origin xyz="0.0 0.22 -0.01" rpy="0 0 0"/>
-        </xacro:link_led>
-    <!-- Green -->
-        <xacro:link_led name="${X_ROBOT_NAMESPACE}/ardrone_green" parent="${X_ROBOT_NAMESPACE}/ardrone_base_link">
-          <origin xyz="-0.22 0.0 -0.01" rpy="0 0 0"/>
-        </xacro:link_led>
 	<gazebo reference="${X_ROBOT_NAMESPACE}/ardrone_base_link">
 		<turnGravityOff>false</turnGravityOff>
 	</gazebo>
-	<gazebo reference="${X_ROBOT_NAMESPACE}/ardrone_red_led">
-		<material>Gazebo/Red</material>
-	</gazebo>
-	<gazebo reference="${X_ROBOT_NAMESPACE}/ardrone_blue_led">
-		<material>Gazebo/Blue</material>
-	</gazebo>
-	<gazebo reference="${X_ROBOT_NAMESPACE}/ardrone_green_led">
-		<material>Gazebo/Green</material>
-	</gazebo>
     <!-- Gazebo Plugins -->
-    <ardrone_plugins/>
+    <usma_ardrone_plugins/>
   </xacro:macro>
 </robot>

File: usma_descriptions/UAV/urdf/usma_ardrone_sensors.urdf.xacro (robot description, xacro)
@@ -1,9 +1,9 @@
-<robot name="ardrone" xmlns:xacro="http://ros.org/wiki/xacro">
+<robot name="usma_ardrone" xmlns:xacro="http://ros.org/wiki/xacro">
     <xacro:property name="M_PI" value="3.1415926535897931" />
-    <xacro:include filename="$(find robot_descriptions)/UAV/urdf/ardrone_base.urdf.xacro" />
+    <xacro:include filename="$(find usma_descriptions)/UAV/urdf/usma_ardrone_base.urdf.xacro" />
     <xacro:property name="X_ROBOT_NAMESPACE" value="/gazebo/uav" />
-    <ardrone_base_macro />
+    <usma_ardrone_base_macro />
     <!-- Sonar height sensor -->
-			<xacro:include filename="$(find robot_descriptions)/UAV/urdf/sensors/sonar_sensor.urdf.xacro" />
+			<xacro:include filename="$(find usma_descriptions)/UAV/urdf/sensors/sonar_sensor.urdf.xacro" />
 			<xacro:sonar_sensor name="ardrone_sonar" parent="${X_ROBOT_NAMESPACE}/ardrone_base_link" ros_topic="ardrone/sonar_height" update_rate="10" min_range="0.01" max_range="3.0" field_of_view="${40*M_PI/180}" ray_count="3">
 				<origin xyz="-0.15 0.0 0.0" rpy="0 ${90*M_PI/180} 0"/>
@@ -16,10 +16,10 @@
     <!-- The following two cameras should be united to one! -->
 	    <!-- Forward facing camera -->
-			<xacro:include filename="$(find robot_descriptions)/UAV/urdf/sensors/generic_camera.urdf.xacro" />
+			<xacro:include filename="$(find usma_descriptions)/UAV/urdf/sensors/generic_camera.urdf.xacro" />
 			<xacro:generic_camera name="front" sim_name="ardrone" parent="${X_ROBOT_NAMESPACE}/ardrone_base_link" update_rate="60" res_x="640" res_y="360" image_format="R8G8B8" hfov="${81*M_PI/180}">
 				<origin xyz="0.21 0.0 0.01" rpy="0 0 0"/>
 			</xacro:generic_camera>
 	    <!-- Downward facing camera -->
-			<xacro:include filename="$(find robot_descriptions)/UAV/urdf/sensors/generic_camera.urdf.xacro" />
+			<xacro:include filename="$(find usma_descriptions)/UAV/urdf/sensors/generic_camera.urdf.xacro" />
 			<xacro:generic_camera name="bottom" sim_name="ardrone" parent="${X_ROBOT_NAMESPACE}/ardrone_base_link" update_rate="60" res_x="640" res_y="360" image_format="R8G8B8" hfov="${81*M_PI/180}">
 				<origin xyz="0.15 0.0 0.0" rpy="0 ${M_PI/2} 0"/>

Commit message: debugging gazebo urdfs

File: usma_descriptions/UAV/urdf/usma_ardrone_base.urdf.xacro (robot description, xacro)
@@ -2,12 +2,11 @@
   <xacro:property name="X_ROBOT_NAMESPACE" value="/gazebo/uav" />
   <xacro:include filename="$(find usma_plugins)/urdf/usma_ardrone_plugins.urdf.xacro" />
-  <!-- Main ardrone link -->
   <xacro:macro name="usma_ardrone_base_macro">
-	<link name="${X_ROBOT_NAMESPACE}/ardrone_base_footprint"/>
-	<joint name="base_joint" type="fixed">
-		<origin xyz="0 0 0.0102" rpy="0 0 0" />
-		<parent link="${X_ROBOT_NAMESPACE}/ardrone_base_footprint"/>
-		<child link="${X_ROBOT_NAMESPACE}/ardrone_base_link" />
-	</joint>
+  	<link name="${X_ROBOT_NAMESPACE}/ardrone_base_footprint"/>
+  	<joint name="base_joint" type="fixed">
+  		<origin xyz="0 0 0.0102" rpy="0 0 0" />
+  		<parent link="${X_ROBOT_NAMESPACE}/ardrone_base_footprint"/>
+  		<child link="${X_ROBOT_NAMESPACE}/ardrone_base_link" />
+  	</joint>
     <link name="${X_ROBOT_NAMESPACE}/ardrone_base_link">
       <inertial>
@@ -19,5 +18,5 @@
         <origin xyz="0 0 0" rpy="0 0 0" />
         <geometry>
-          <mesh filename="package://robot_descriptions/UAV/meshes/ardrone_4.dae"/>
+          <mesh filename="package://usma_descriptions/UAV/meshes/ardrone_4.dae"/>
         </geometry>
       </visual>
@@ -25,5 +24,5 @@
         <origin xyz="0 0 0" rpy="0 0 0" />
         <geometry>
-          <mesh filename="package://robot_descriptions/UAV/meshes/ardrone_4.stl"/>
+          <mesh filename="package://usma_descriptions/UAV/meshes/ardrone_4.stl"/>
         </geometry>
       </collision>

File: usma_descriptions/UAV/urdf/usma_ardrone_rviz_base.urdf.xacro (robot description, xacro)
@@ -1,14 +1,5 @@
-<robot name="usma_ardrone_rviz" xmlns:xacro="http://ros.org/wiki/xacro">
+<robot name="usma_ardrone_rviz_base" xmlns:xacro="http://ros.org/wiki/xacro">
 	<xacro:property name="X_ROBOT_NAMESPACE" value="/vicon/uav" />
-	<!-- Main ardrone link -->
 	<xacro:macro name="usma_ardrone_rviz_macro">
-<!-- 		<link name="${X_ROBOT_NAMESPACE}/base_footprint"/>
-		<joint name="base_joint" type="fixed">
-			<origin xyz="0 0 0" rpy="0 0 0" />
-			<parent link="${X_ROBOT_NAMESPACE}/base_footprint"/>
-			<child link="${X_ROBOT_NAMESPACE}/base_link" />
-		</joint>
-		<link name="${X_ROBOT_NAMESPACE}/base_link">
- -->
 		<link name="${X_ROBOT_NAMESPACE}/base_footprint">
  			<inertial>

File: usma_plugins/urdf/usma_ardrone_plugins.urdf.xacro (robot description, xacro)
@@ -7,6 +7,6 @@
 	<xacro:macro name="usma_ardrone_plugins">
 		<canonicalBody>${X_ROBOT_NAMESPACE}/ardrone_base_link</canonicalBody>
-		<ardrone_sensors/>
-		<ardrone_controller/>
+		<usma_ardrone_sensors/>
+		<usma_ardrone_controller/>
 	</xacro:macro>
 </robot>

File: usma_plugins/urdf/usma_ardrone_simple_controller.urdf.xacro (robot description, xacro)
@@ -5,6 +5,5 @@
     <xacro:macro name="usma_ardrone_controller">
         <gazebo>
-            <plugin name="ardrone_simple_controller" filename="libusma_ardrone_simple_controller.so">
-            <!-- <plugin name="ardrone_simple_controller" filename="libhector_gazebo_quadrotor_simple_controller.so"> -->
+            <plugin name="usma_ardrone_simple_controller" filename="libusma_ardrone_simple_controller.so">
                 <alwaysOn>true</alwaysOn>
                 <updateRate>0.0</updateRate>
