Commit message: fixed issue with robot_descriptions vs usma_descriptions

File: usma_descriptions/UAV/urdf/sensors/hokuyo_utm30lx.urdf.xacro (robot description, xacro)
@@ -15,5 +15,5 @@
 	  <origin xyz="0 0 0" rpy="0 0 0" />
           <geometry>
-          <mesh filename="package://robot_descriptions/common/meshes/hokuyo_utm30lx/hokuyo_utm_30lx$(optenv TEST_SELF_FILTER).dae"/>
+          <mesh filename="package://usma_descriptions/common/meshes/hokuyo_utm30lx/hokuyo_utm_30lx$(optenv TEST_SELF_FILTER).dae"/>
         </geometry>
 	</visual>

File: usma_descriptions/UAV/urdf/sensors/sonar_sensor.urdf.xacro (robot description, xacro)
@@ -16,5 +16,5 @@
         <geometry>
           <!--<box size="0.01 0.01 0.01" /> -->
-          <mesh filename="package://robot_descriptions/common/meshes/sonar_sensor/max_sonar_ez4.dae"/>
+          <mesh filename="package://usma_descriptions/common/meshes/sonar_sensor/max_sonar_ez4.dae"/>
         </geometry>
       </visual>

File: usma_descriptions/UAV/urdf/usma_ardrone_rviz.urdf.xacro (robot description, xacro)
@@ -1,4 +1,4 @@
 <robot name="usma_ardrone_rviz" xmlns:xacro="http://ros.org/wiki/xacro">
-    <xacro:include filename="$(find robot_descriptions)/UAV/urdf/usma_ardrone_rviz_base.urdf.xacro" />
+    <xacro:include filename="$(find usma_descriptions)/UAV/urdf/usma_ardrone_rviz_base.urdf.xacro" />
     <usma_ardrone_rviz_macro />
 </robot>

File: usma_plugins/urdf/usma_ardrone_simple_controller.urdf.xacro (robot description, xacro)
@@ -12,6 +12,6 @@
                 <imuTopic>ardrone/imu</imuTopic>
                 <topicName>usma_ardrone/uav/cmd_vel</topicName>
-                <mocapBodyName>/vrpn_client_node/parrot/pose</mocapBodyName>
-                <mocapPoseTopic>/vrpn_client_node/parrot/pose</mocapPoseTopic>
+                <mocapBodyName>/vrpn_client_node/Ardrone2/pose</mocapBodyName>
+                <mocapPoseTopic>/vrpn_client_node/Ardrone2/pose</mocapPoseTopic>
                 <!-- /vrpn_client_node/parrot/pose -->
                 <mocapOriginName>/mocap/origin</mocapOriginName>
